Commit message: [fix] change stl file path to include stl file properly

File: pa10_description/urdf/pa10.xacro (robot description, xacro)
@@ -15,5 +15,5 @@
       <origin rpy="0 0 3.14" xyz="0 0 0"/>
       <geometry>
-        <mesh filename="file:///home/ubuntin/pa10_stl/S1.stl"/>
+        <mesh filename="file://$(find pa10_stl)/S1.stl"/>
 <!-- podemos usar tambien en vez de mesh que requiere un archivo, cilindros cajas o esferas!!! -->
       </geometry>
@@ -25,5 +25,5 @@
       <origin rpy="0 0 3.14" xyz="0 0 0"/>
       <geometry>
-        <mesh filename="file:///home/ubuntin/pa10_stl_collision/S1_collision.stl"/>
+        <mesh filename="file://$(find pa10_stl_collision)/S1_collision.stl"/>
       </geometry>
     </collision>
@@ -41,5 +41,5 @@
       <origin rpy="0 0 0" xyz="0 0 0.117"/>
       <geometry>
-        <mesh filename="file:///home/ubuntin/pa10_stl/S2.stl"/>
+        <mesh filename="file://$(find pa10_stl)/S2.stl"/>
       </geometry>
 	<material name="">
@@ -50,5 +50,5 @@
       <origin rpy="0 0 0" xyz="0 0 0.117"/>
       <geometry>
-        <mesh filename="file:///home/ubuntin/pa10_stl_collision/S2_collision.stl"/>
+        <mesh filename="file://$(find pa10_stl_collision)/S2_collision.stl"/>
       </geometry>
     </collision>
@@ -66,5 +66,5 @@
       <origin rpy="0 0 0" xyz="0 0 0"/>
       <geometry>
-        <mesh filename="file:///home/ubuntin/pa10_stl/S3.stl"/>
+        <mesh filename="file://$(find pa10_stl)/S3.stl"/>
       </geometry>
       <material name="">
@@ -75,5 +75,5 @@
       <origin rpy="0 0 0" xyz="0 0 0"/>
       <geometry>
-        <mesh filename="file:///home/ubuntin/pa10_stl_collision/S3_collision.stl"/>
+        <mesh filename="file://$(find pa10_stl_collision)/S3_collision.stl"/>
       </geometry>
     </collision>
@@ -91,5 +91,5 @@
       <origin rpy="0 0 0" xyz="0 0 0.133"/>
       <geometry>
-        <mesh filename="file:///home/ubuntin/pa10_stl/E1.stl"/>
+        <mesh filename="file://$(find pa10_stl)/E1.stl"/>
       </geometry>
 	<material name="">
@@ -100,5 +100,5 @@
       <origin rpy="0 0 0" xyz="0 0 0.133"/>
       <geometry>
-        <mesh filename="file:///home/ubuntin/pa10_stl_collision/E1_collision.stl"/>
+        <mesh filename="file://$(find pa10_stl_collision)/E1_collision.stl"/>
       </geometry>
     </collision>
@@ -116,5 +116,5 @@
       <origin rpy="0 0 0" xyz="0 0.003 0"/>
       <geometry>
-        <mesh filename="file:///home/ubuntin/pa10_stl/E2.stl"/>
+        <mesh filename="file://$(find pa10_stl)/E2.stl"/>
       </geometry>
 	<material name="">
@@ -125,5 +125,5 @@
       <origin rpy="0 0 0" xyz="0 0.003 0"/>
       <geometry>
-        <mesh filename="file:///home/ubuntin/pa10_stl_collision/E2_collision.stl"/>
+        <mesh filename="file://$(find pa10_stl_collision)/E2_collision.stl"/>
       </geometry>
     </collision>
@@ -141,5 +141,5 @@
       <origin rpy="0 0 0" xyz="0 0 0.195"/>
       <geometry>
-        <mesh filename="file:///home/ubuntin/pa10_stl/W1.stl"/>
+        <mesh filename="file://$(find pa10_stl)/W1.stl"/>
       </geometry>
 	<material name="">
@@ -150,5 +150,5 @@
       <origin rpy="0 0 0" xyz="0 0 0.195"/>
       <geometry>
-        <mesh filename="file:///home/ubuntin/pa10_stl_collision/W1_collision.stl"/>
+        <mesh filename="file://$(find pa10_stl_collision)/W1_collision.stl"/>
       </geometry>
     </collision>
@@ -166,14 +166,14 @@
       <origin rpy="0 0 0" xyz="0 0 0"/>
       <geometry>
-        <mesh filename="file:///home/ubuntin/pa10_stl/W2.stl"/>
-      </geometry>
-	<material name="">
-        <color rgba="0.34 0.35 0.36 1.0"/>
-      </material>
-    </visual>
-    <collision>
-      <origin rpy="0 0 0" xyz="0 0 0"/>
-      <geometry>
-        <mesh filename="file:///home/ubuntin/pa10_stl_collision/W2_collision.stl"/>
+        <mesh filename="file://$(find pa10_stl)/W2.stl"/>
+      </geometry>
+	<material name="">
+        <color rgba="0.34 0.35 0.36 1.0"/>
+      </material>
+    </visual>
+    <collision>
+      <origin rpy="0 0 0" xyz="0 0 0"/>
+      <geometry>
+        <mesh filename="file://$(find pa10_stl_collision)/W2_collision.stl"/>
       </geometry>
     </collision>
